File: pcb/_autosave-hola.sch (KiCad schematic (older format))
At the start: 35 parts, among them J1 USB_B, J2 USB_B_Micro, J3 Conn_01x08_Female, J4 Conn_01x02, Q1 DTB123T, U1 TPS61090, U2 MCP73871

Commit message: avance 23-09-2021
Parts:
- removed J3: Conn_01x08_Female, Connector_Harwin:Harwin_M20-89008xx_1x08_P2.54mm_Horizontal, symbol Connector:Conn_01x08_Female
- added J3: Conn_01x08, Connector_Hirose:Hirose_DF13-08P-1.25DSA_1x08_P1.25mm_Vertical, symbol Connector_Generic:Conn_01x08
Connections:
- net +5V: now also J3.8 (Pin_8); no longer C1.1, C2.1, L1.1, Q1.2 (E), R1.2, R15.2, U1.8 (VBAT)
- net +BATT: now also C1.1, C2.1, L1.1, Q1.2 (E), R1.2, R15.2, U1.8 (VBAT), J3.2 (Pin_2)
- net +VSW: now also J3.3 (Pin_3)
- net GND: now also J3.7 (Pin_7)
- net VBUS: now also J3.1 (Pin_1)
Other:
- note added: "Boost converter"
- note added: "Circuito Li-ion"
- note added: "Circuito USB"
- note removed: "hola amigo"
- moved on the sheet: C5, J1, J2, R3, R4, R5, R6
