File: pcb/hola.sch (KiCad schematic (older format))
At the start: 32 parts, among them J1 USB_B, J2 USB_B_Micro, Q1 DTB123T, U1 TPS61090, U2 MCP73871

Commit message: avance 23-09-2021
Parts:
- added D4: LED, LED_THT:LED_D8.0mm, symbol Device:LED
- added J4: Conn_01x02, Connector:Banana_Jack_2Pin, symbol Connector_Generic:Conn_01x02
- added R16: 1k, Resistor_SMD:R_MELF_MMB-0207, symbol Device:R
- BT1: footprint (none) -> Battery:BatteryHolder_Keystone_104_1x23mm
- C1: value CAP -> 10uF; footprint (none) -> Capacitor_THT:C_Disc_D3.8mm_W2.6mm_P2.50mm
- C2: value CAP -> 0.1uF; footprint (none) -> Capacitor_THT:C_Disc_D3.8mm_W2.6mm_P2.50mm
- C3: value CAP -> 2.2uF; footprint (none) -> Capacitor_THT:C_Disc_D3.8mm_W2.6mm_P2.50mm
- C4: value CP1 -> 100uF; footprint (none) -> Capacitor_THT:C_Disc_D3.8mm_W2.6mm_P2.50mm
- C5, C6: footprint (none) -> Capacitor_THT:C_Disc_D3.8mm_W2.6mm_P2.50mm
- D1, D2, D3: footprint (none) -> LED_THT:LED_D8.0mm
- J1: footprint (none) -> Connector_USB:USB_B_Amphenol_MUSB-D511_Vertical_Rugged
- J2: footprint (none) -> Connector_USB:USB_Micro-B_Amphenol_10103594-0001LF_Horizontal
- J3: renamed from J?; footprint (none) -> Connector_Harwin:Harwin_M20-89008xx_1x08_P2.54mm_Horizontal
- L1: value INDUCTOR -> 6.4uH; footprint (none) -> Inductor_THT:L_Axial_L12.8mm_D5.8mm_P20.32mm_Horizontal_Fastron_HBCC
- Q1: footprint (none) -> OptoDevice:Vishay_MINIMOLD-3Pin
- R1: value R -> 1.87M; footprint (none) -> Resistor_SMD:R_MELF_MMB-0207
- R10: value R -> 270k; footprint (none) -> Resistor_SMD:R_MELF_MMB-0207
- R11: value R -> 100k; footprint (none) -> Resistor_SMD:R_MELF_MMB-0207
- R12: footprint (none) -> Resistor_SMD:R_MELF_MMB-0207
- R13, R14, R9: value R -> 1k; footprint (none) -> Resistor_SMD:R_MELF_MMB-0207
- R15: renamed from R?; value R -> 200k; footprint (none) -> Resistor_SMD:R_MELF_MMB-0207
- R2: value R -> 310k; footprint (none) -> Resistor_SMD:R_MELF_MMB-0207
- R3: value R -> 43k; footprint (none) -> Resistor_SMD:R_MELF_MMB-0207
- R4: value R -> 49.9k; footprint (none) -> Resistor_SMD:R_MELF_MMB-0207
- R5: value R -> 5k; footprint (none) -> Resistor_SMD:R_MELF_MMB-0207
- R6: value R -> 9.9k; footprint (none) -> Resistor_SMD:R_MELF_MMB-0207
- R7: value R -> 1.07M; footprint (none) -> Resistor_SMD:R_MELF_MMB-0207
- R8: value R -> 200k; footprint (none) -> Resistor_SMD:R_MELF_MMB-0207
Connections:
- net labels added: +BATT, +VSW, VBUS
- wire segments 131 -> 146
- no-connect marks 0 -> 12
Other:
- moved on the sheet: C3, C4, D1, Q1, R3, R6, R7, R8, R9

Commit message: avance 23-09-2021
Parts:
- removed J3: Conn_01x08_Female, Connector_Harwin:Harwin_M20-89008xx_1x08_P2.54mm_Horizontal, symbol Connector:Conn_01x08_Female
- added J3: Conn_01x08, Connector_Hirose:Hirose_DF13-08P-1.25DSA_1x08_P1.25mm_Vertical, symbol Connector_Generic:Conn_01x08
Other:
- note added: "Boost converter"
- note added: "Circuito Li-ion"
- note added: "Circuito USB"
- moved on the sheet: BT1, C1, C2, C3, C4, C5, C6, D1, D2, D3, D4, J1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

Commit message: TP Final
Parts:
- BT1: footprint Battery:BatteryHolder_Keystone_104_1x23mm -> Battery:BatteryHolder_Keystone_3000_1x12mm
- C1, C2, C3, C4, C5, C6: footprint Capacitor_THT:C_Disc_D3.8mm_W2.6mm_P2.50mm -> Capacitor_SMD:C_0402_1005Metric_Pad0.74x0.62mm_HandSolder
- D1, D2, D3, D4: footprint LED_THT:LED_D8.0mm -> LED_SMD:LED_2010_5025Metric_Castellated
- J4: footprint Connector:Banana_Jack_2Pin -> Connector:JWT_A3963_1x02_P3.96mm_Vertical
- L1: footprint Inductor_THT:L_Axial_L12.8mm_D5.8mm_P20.32mm_Horizontal_Fastron_HBCC -> Inductor_SMD:L_1806_4516Metric
- Q1: footprint OptoDevice:Vishay_MINIMOLD-3Pin -> Package_TO_SOT_SMD:SOT-23_Handsoldering
- R1, R10, R11, R12, R13, R14, R15, R16, R2, R3, R4, R5, R6, R7, R8, R9: footprint Resistor_SMD:R_MELF_MMB-0207 -> Resistor_SMD:R_1206_3216Metric
Connections:
- net +5V: no longer C1.1, C2.1, L1.1, Q1.2 (E), R1.2, R15.2, U1.8 (VBAT)
- net +BATT: now also C1.1, C2.1, L1.1, Q1.2 (E), R1.2, R15.2, U1.8 (VBAT)
Other:
- note added: "in"
- note added: "out"
- moved on the sheet: C5, J1, J2, R3, R4, R5, R6

Commit message: actualizacion
Parts:
- added H1, H2, H3, H4: MountingHole, MountingHole:MountingHole_2.1mm, symbol Mechanical:MountingHole
Changed lines of the file:
@@
 Wire Wire Line
 	8100 3900 8100 4300
+$Comp
+L Mechanical:MountingHole H1
+U 1 1 61700954
+P 6950 5250
+F 0 "H1" H 7050 5296 50  0000 L CNN
+F 1 "MountingHole" H 7050 5205 50  0000 L CNN
+F 2 "MountingHole:MountingHole_2.1mm" H 6950 5250 50  0001 C CNN
+F 3 "~" H 6950 5250 50  0001 C CNN
+	1    6950 5250
+	1    0    0    -1
+$EndComp
+$Comp
+L Mechanical:MountingHole H2
+U 1 1 617012D8
+P 6950 5500
+F 0 "H2" H 7050 5546 50  0000 L CNN
+F 1 "MountingHole" H 7050 5455 50  0000 L CNN
+F 2 "MountingHole:MountingHole_2.1mm" H 6950 5500 50  0001 C CNN
+F 3 "~" H 6950 5500 50  0001 C CNN
+	1    6950 5500
+	1    0    0    -1
+$EndComp
+$Comp
+L Mechanical:MountingHole H3
+U 1 1 61701D3B
+P 6950 5750
+F 0 "H3" H 7050 5796 50  0000 L CNN
+F 1 "MountingHole" H 7050 5705 50  0000 L CNN
+F 2 "MountingHole:MountingHole_2.1mm" H 6950 5750 50  0001 C CNN
+F 3 "~" H 6950 5750 50  0001 C CNN
+	1    6950 5750
+	1    0    0    -1
+$EndComp
+$Comp
+L Mechanical:MountingHole H4
+U 1 1 61702385
+P 6950 6000
+F 0 "H4" H 7050 6046 50  0000 L CNN
+F 1 "MountingHole" H 7050 5955 50  0000 L CNN
+F 2 "MountingHole:MountingHole_2.1mm" H 6950 6000 50  0001 C CNN
+F 3 "~" H 6950 6000 50  0001 C CNN
+	1    6950 6000
+	1    0    0    -1
+$EndComp
 $EndSCHEMATC

Commit message: actualizacion
Parts:
- removed BT1: Battery_Cell, Battery:BatteryHolder_Keystone_3000_1x12mm, symbol Device:Battery_Cell
- added J5: Conn_01x02, Connector_JST:JST_PH_S2B-PH-K_1x02_P2.00mm_Horizontal, symbol Connector_Generic:Conn_01x02
Connections:
- net +VSW: now also J5.1 (Pin_1)
- net GND: now also J5.2 (Pin_2)
Changed lines of the file:
@@
-$EndComp
-$Comp
-L Device:Battery_Cell BT1
-U 1 1 6146719E
-P 10300 3250
-F 0 "BT1" H 10418 3346 50  0000 L CNN
-F 1 "Battery_Cell" H 10418 3255 50  0000 L CNN
-F 2 "Battery:BatteryHolder_Keystone_3000_1x12mm" V 10300 3310 50  0001 C CNN
-F 3 "https://www.mouser.com/Power/Battery-Holders-Clips-Contacts/Datasheets/_/N-cicxg?keyword=534-104" V 10300 3310 50  0001 C CNN
-	1    10300 3250
-	1    0    0    -1
 $EndComp
 $Comp
@@
 $EndComp
 Wire Wire Line
-	10300 3350 10300 3750
-Wire Wire Line
 	9850 3450 9850 3750
-Wire Wire Line
-	10300 3050 10300 2700
-Wire Wire Line
-	10300 2700 9850 2700
 Wire Wire Line
 	9850 2700 9850 2950
@@
 	1    0    0    -1
 $EndComp
+$Comp
+L Connector_Generic:Conn_01x02 J5
+U 1 1 6172C34A
+P 10550 3150
+F 0 "J5" H 10630 3142 50  0000 L CNN
+F 1 "Conn_01x02" H 10630 3051 50  0000 L CNN
+F 2 "Connector_JST:JST_PH_S2B-PH-K_1x02_P2.00mm_Horizontal" H 10550 3150 50  0001 C CNN
+F 3 "~" H 10550 3150 50  0001 C CNN
+	1    10550 3150
+	1    0    0    -1
+$EndComp
+Wire Wire Line
+	10300 3750 10300 3250
+Wire Wire Line
+	10300 3250 10350 3250
+Wire Wire Line
+	10350 3150 10300 3150
+Wire Wire Line
+	10300 3150 10300 2700
+Wire Wire Line
+	10300 2700 9850 2700
 $EndSCHEMATC
